File: pcb_design/TR108 Mainboard/TR108 Mainboard.kicad_pcb (KiCad board)
At the start: 2 copper layers, 69.8 x 97.7 mm, 17 parts, among them J1 Raspberry Pi Zero, J2 Sense Hat, J3 power connector, J4 front panel connector, J5 Composite Video, J6 Conn_01x08_Female

Commit message: Update to PCB
Parts:
- added J3: i2c Expansion, Connector_PinHeader_2.54mm:PinHeader_1x04_P2.54mm_Vertical, F.Cu at (138.1, 49.2)
- added J7: i2c Expansion, Connector_PinHeader_2.54mm:PinHeader_1x04_P2.54mm_Vertical, F.Cu at (104.2, 121.5)
- added JP8: SolderJumper_2_Open, Jumper:SolderJumper-2_P1.3mm_Open_RoundedPad1.0x1.5mm, F.Cu at (187.7, 87.0)
- added U1: 74HC595, Package_SO:SOIC-16_3.9x9.9mm_P1.27mm, F.Cu at (138.7, 108.2)
- moved JP1 9.47 mm to (120.3, 66.4)
- moved JP2 9.46 mm to (120.3, 68.8)
- moved JP3 9.45 mm to (120.3, 71.2)
- moved G*** 3.67 mm to (134.3, 120.0)
- renumbered J6 to J4, J4 to J5, J3 to J6, J5 to J8, JP3 to JP2, JP2 to JP3, JP7 to JP4, JP6 to JP5, JP4 to JP6, JP5 to JP7
Routing:
- net SCL: track 33.3 -> 166.0 mm, vias 0 -> 5
- net SDA: track 30.8 -> 152.8 mm, vias 0 -> 4
- net SC_CS: track 5.80 -> 15.9 mm
- net 8: track 101.2 -> 91.3 mm
- net SC_RESET: track 6.00 -> 15.8 mm
- net 24: track 95.3 -> 85.5 mm
- net SC_A0: track 6.00 -> 15.8 mm
- net 23: track 97.5 -> 87.7 mm
- net Net-(J1-Pad7): vias 0 -> 2
Other:
- board size 69.8 x 97.7 mm -> 69 x 98 mm
- board text added: "5V"
- board text added: "BACKPLANE - REV 1"
- board text added: "CB 2021 - LIVE LONG AND PROSPER"
- board text added: "GNDN"
- board text added: "I2C EXPANSION"
- board text added: "POWER INTERLINK"
- board text added: "RASPBERRY PI ZERO"
- board text added: "SCL"
- board text added: "SCREEN MODULE"
- board text added: "ST7735 Screen"
- board text added: "TR-108 PICORDER"
- board text added: "“3v3”"
- board text added: "“A0”"
- board text added: "“CS”"
- board text added: "“GND”"
- board text added: "“LED”"
- board text added: "“RST”"
- board text added: "“SCK”"
- board text added: "“SDA”"
- board text removed: "5V in"
- board text removed: "A0"
- board text removed: "CS"
- board text removed: "LED"
- board text removed: "RST"
- board text removed: "Raspberry Pi Zero"
- board text removed: "SCK"
- board text removed: "TR-108 PICORDER BACKPLANE - REV 1"

Commit message: mass update - new blend and pcb
Parts:
- removed JP4, JP5, JP6, JP7, JP8: SolderJumper_2_Open, Jumper:SolderJumper-2_P1.3mm_Open_RoundedPad1.0x1.5mm
- removed U1: 74HC595, Package_SO:SOIC-16_3.9x9.9mm_P1.27mm
- added J10: PG GPIO, Connector_PinHeader_2.54mm:PinHeader_1x04_P2.54mm_Vertical, F.Cu at (154.4, 49.2)
- added J9: Audio Out, Connector_PinHeader_2.54mm:PinHeader_1x03_P2.54mm_Vertical, F.Cu at (117.5, 138.6)
- added REF**: MountingHole_2.2mm_M2, MountingHole:MountingHole_2.2mm_M2, F.Cu at (164.9, 49.1)
- added REF**: MountingHole_2.2mm_M2, MountingHole:MountingHole_2.2mm_M2, F.Cu at (104.3, 49.1)
- added REF**: MountingHole_2.2mm_M2, MountingHole:MountingHole_2.2mm_M2, F.Cu at (104.3, 138.7)
- added REF**: MountingHole_2.2mm_M2, MountingHole:MountingHole_2.2mm_M2, F.Cu at (164.9, 138.8)
- R1, R2, R3: footprint Resistor_SMD:R_0603_1608Metric_Pad0.98x0.95mm_HandSolder -> Resistor_SMD:R_0805_2012Metric_Pad1.20x1.40mm_HandSolder
- moved R2 34.1 mm to (113.2, 69.5)
- moved R3 34.1 mm to (113.2, 72.1)
- moved R1 31.9 mm to (113.1, 67.0)
- moved J4 25.0 mm to (104.2, 85.2)
- moved JP3 24.1 mm to (119.3, 95.4)
- moved JP2 24.0 mm to (119.3, 92.8)
- moved JP1 23.9 mm to (119.3, 90.3)
- moved J5 23.0 mm to (104.2, 59.4)
- moved G*** 1.70 mm to (134.3, 121.7)
Connections:
- J1 pad 27: Net-(J1-Pad27) -> ID_SD
- J1 pad 28: Net-(J1-Pad28) -> ID_SC
- J1 pad 32: Net-(J1-Pad32) -> audio1
- J1 pad 33: button3 -> audio2
- J1 pad 36: Net-(J1-Pad36) -> button3
- J1 pad 38: Net-(J1-Pad38) -> SIG
- J1 pad 40: Net-(J1-Pad40) -> NS
- J2 pad 16: Net-(J2-Pad16) -> 23
- J2 pad 18: Net-(J2-Pad18) -> 24
- J2 pad 22: Net-(J2-Pad22) -> 25
- J2 pad 24: Net-(J2-Pad24) -> 8
- J2 pad 27: Net-(J2-Pad27) -> ID_SD
- J2 pad 28: Net-(J2-Pad28) -> ID_SC
- J6 pad 3: Net-(J6-Pad3) -> GND
Routing:
- net NS: track 0.00 -> 101.2 mm, vias 0 -> 1
- net SIG: track 0.00 -> 94.8 mm, vias 0 -> 1
- net ID_SC: track 0.00 -> 87.3 mm, vias 0 -> 3
- net ID_SD: track 0.00 -> 86.7 mm, vias 0 -> 3
- net audio1: track 0.00 -> 58.2 mm, vias 0 -> 2
- net audio2: track 0.00 -> 54.8 mm, vias 0 -> 2
- net Net-(J1-Pad11): track 29.0 -> 74.2 mm, vias 0 -> 2
- net Net-(J1-Pad13): track 28.9 -> 73.7 mm, vias 0 -> 2
- net Net-(J1-Pad7): track 29.0 -> 71.8 mm
- net Net-(J2-Pad18): track 36.0 -> 0.00 mm
- net button3: track 79.7 -> 107.1 mm
- net SC_SCK: track 93.9 -> 69.1 mm, vias 3 -> 2
- net 6V: track 38.9 -> 63.5 mm
- net GND: track 0.00 -> 24.5 mm
- net VIDEO: track 93.2 -> 117.6 mm
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Other:
- outline, holes or cut-outs redrawn
- net class Default removed
- board text added: "A1 (12)"
- board text added: "A2 (13)"
- board text added: "BACKPLANE - REV 2"
- board text added: "CB 2022 - LIVE LONG AND PROSPER"
- board text added: "LUMA SCREEN"
- board text added: "NS (21)"
- board text added: "PG RADIATION"
- board text added: "PWM AUDIO"
- board text added: "SIG (20)"
- board text added: "“A0” (23)"
- board text added: "“CS” (8)"
- board text added: "“LED” (15)"
- board text added: "“RST” (24)"
- board text added: "“SCK” (23)"
- board text added: "“SDA” (10)"
- board text removed: "BACKPLANE - REV 1"
- board text removed: "CB 2021 - LIVE LONG AND PROSPER"
- board text removed: "ST7735 Screen"
- board text removed: "TR-108 PICORDER"
- board text removed: "“A0”"
- board text removed: "“CS”"
- board text removed: "“LED”"
- board text removed: "“RST”"
- board text removed: "“SCK”"
- board text removed: "“SDA”"
