File: pcb_design/TR108 Mainboard/TR108 Mainboard.sch (KiCad schematic (older format))
At the start: 16 parts, among them J1 Raspberry Pi Zero, J2 Sense Hat, J3 power connector, J4 front panel connector, J5 Composite Video, J6 Conn_01x08_Female

Commit message: Update to PCB
Parts:
- added J3, J7: i2c Expansion, Connector_PinHeader_2.54mm:PinHeader_1x04_P2.54mm_Vertical, symbol Connector:Conn_01x04_Female
- added JP10, JP8, JP9: SolderJumper_2_Open, Jumper:SolderJumper-2_P1.3mm_Open_RoundedPad1.0x1.5mm, symbol Jumper:SolderJumper_2_Open
- added U1: 74HC595, Package_SO:SOIC-16_3.9x9.9mm_P1.27mm, symbol 74xx:74HC595
- renumbered J6 to J4, J4 to J5, J3 to J6, J5 to J8, JP3 to JP2, JP2 to JP3, JP7 to JP4, JP6 to JP5, JP4 to JP6, JP5 to JP7
Connections:
- net 3v3: now also J3.2 (Pin_2), J7.2 (Pin_2)
- net 5V: now also U1.10 (~SRCLR), U1.16 (VCC)
- net GND: now also J3.3 (Pin_3), J7.3 (Pin_3), U1.13 (~OE), U1.8 (GND)
- net SCL: now also J3.4 (Pin_4), J7.4 (Pin_4)
- net SDA: now also J3.1 (Pin_1), J7.1 (Pin_1)
- net shift_serial: now reaches J1.7 (GCLK0/GPIO4), R1.2
- net shift_serial: now also JP8.1 (A)
- new net: JP9.2 (B), U1.11 (SRCLK)
- new net: JP10.2 (B), U1.12 (RCLK)
- new net: JP8.2 (B), U1.14 (SER)
- new net shift_clock: JP9.1 (A)
Changed lines of the file:
@@
 LED3
 $Comp
-L Connector:Conn_01x09_Female J4
+L Connector:Conn_01x09_Female J5
 U 1 1 6025E134
 P 3800 5150
-F 0 "J4" H 3828 5126 50  0000 L CNN
+F 0 "J5" H 3828 5126 50  0000 L CNN
 F 1 "front panel connector" H 3828 5035 50  0000 L CNN
 F 2 "Connector_PinHeader_2.54mm:PinHeader_1x09_P2.54mm_Vertical" H 3800 5150 50  0001 C CNN
@@
 GND
 $Comp
-L Connector:Conn_01x04_Female J3
+L Connector:Conn_01x04_Female J6
 U 1 1 60261DCC
 P 3450 6400
-F 0 "J3" H 3478 6376 50  0000 L CNN
+F 0 "J6" H 3478 6376 50  0000 L CNN
 F 1 "power connector" H 3478 6285 50  0000 L CNN
 F 2 "Connector_PinHeader_2.54mm:PinHeader_1x04_P2.54mm_Vertical" H 3450 6400 50  0001 C CNN
@@
 VIDEO
 $Comp
-L Connector:Conn_01x02_Female J5
+L Connector:Conn_01x02_Female J8
 U 1 1 60681490
 P 5800 5900
-F 0 "J5" H 5828 5876 50  0000 L CNN
+F 0 "J8" H 5828 5876 50  0000 L CNN
 F 1 "Composite Video" H 5828 5785 50  0000 L CNN
 F 2 "Connector_PinHeader_2.54mm:PinHeader_1x02_P2.54mm_Vertical" H 5800 5900 50  0001 C CNN
@@
 24
 $Comp
-L Jumper:SolderJumper_2_Open JP4
+L Jumper:SolderJumper_2_Open JP6
 U 1 1 60C07218
 P 7000 3050
-F 0 "JP4" H 7000 3255 50  0000 C CNN
+F 0 "JP6" H 7000 3255 50  0000 C CNN
 F 1 "SolderJumper_2_Open" H 7000 3164 50  0000 C CNN
 F 2 "Jumper:SolderJumper-2_P1.3mm_Open_RoundedPad1.0x1.5mm" H 7000 3050 50  0001 C CNN
@@
 	7150 3050 7900 3050
 $Comp
-L Jumper:SolderJumper_2_Open JP5
+L Jumper:SolderJumper_2_Open JP7
 U 1 1 60C08660
 P 7000 3150
-F 0 "JP5" H 7000 3355 50  0000 C CNN
+F 0 "JP7" H 7000 3355 50  0000 C CNN
 F 1 "SolderJumper_2_Open" H 7000 3264 50  0000 C CNN
 F 2 "Jumper:SolderJumper-2_P1.3mm_Open_RoundedPad1.0x1.5mm" H 7000 3150 50  0001 C CNN
@@
 	7900 3150 7150 3150
 $Comp
-L Jumper:SolderJumper_2_Open JP6
+L Jumper:SolderJumper_2_Open JP5
 U 1 1 60C09276
 P 7000 3250
-F 0 "JP6" H 7000 3455 50  0000 C CNN
+F 0 "JP5" H 7000 3455 50  0000 C CNN
 F 1 "SolderJumper_2_Open" H 7000 3364 50  0000 C CNN
 F 2 "Jumper:SolderJumper-2_P1.3mm_Open_RoundedPad1.0x1.5mm" H 7000 3250 50  0001 C CNN
@@
 	7150 3250 7900 3250
 $Comp
-L Jumper:SolderJumper_2_Open JP7
+L Jumper:SolderJumper_2_Open JP4
 U 1 1 60C09F44
 P 9650 2950
-F 0 "JP7" H 9650 3155 50  0000 C CNN
+F 0 "JP4" H 9650 3155 50  0000 C CNN
 F 1 "SolderJumper_2_Open" H 9650 3064 50  0000 C CNN
 F 2 "Jumper:SolderJumper-2_P1.3mm_Open_RoundedPad1.0x1.5mm" H 9650 2950 50  0001 C CNN
@@
 24
 $Comp
-L Connector:Conn_01x08_Female J6
+L Connector:Conn_01x08_Female J4
 U 1 1 60C20AA0
 P 6100 4400
-F 0 "J6" H 6128 4376 50  0000 L CNN
+F 0 "J4" H 6128 4376 50  0000 L CNN
 F 1 "Conn_01x08_Female" H 6128 4285 50  0000 L CNN
 F 2 "Connector_PinHeader_2.54mm:PinHeader_1x08_P2.54mm_Vertical" H 6100 4400 50  0001 C CNN
@@
 23
 $Comp
-L Jumper:SolderJumper_2_Open JP2
+L Jumper:SolderJumper_2_Open JP3
 U 1 1 60C235F4
 P 5350 3350
-F 0 "JP2" H 5350 3125 50  0000 C CNN
+F 0 "JP3" H 5350 3125 50  0000 C CNN
 F 1 "SolderJumper_2_Open" H 5350 3216 50  0000 C CNN
 F 2 "Jumper:SolderJumper-2_P1.3mm_Open_RoundedPad1.0x1.5mm" H 5350 3350 50  0001 C CNN
@@
 SC_RESET
 $Comp
-L Jumper:SolderJumper_2_Open JP3
+L Jumper:SolderJumper_2_Open JP2
 U 1 1 60C23FF2
 P 5350 3550
-F 0 "JP3" H 5350 3325 50  0000 C CNN
+F 0 "JP2" H 5350 3325 50  0000 C CNN
 F 1 "SolderJumper_2_Open" H 5350 3416 50  0000 C CNN
 F 2 "Jumper:SolderJumper-2_P1.3mm_Open_RoundedPad1.0x1.5mm" H 5350 3550 50  0001 C CNN
@@
 Text GLabel 3250 6600 0    50   Input ~ 0
 6V
+$Comp
+L Connector:Conn_01x04_Female J7
+U 1 1 60D031EC
+P 8250 5300
+F 0 "J7" H 8278 5276 50  0000 L CNN
+F 1 "i2c Expansion" H 8278 5185 50  0000 L CNN
+F 2 "Connector_PinHeader_2.54mm:PinHeader_1x04_P2.54mm_Vertical" H 8250 5300 50  0001 C CNN
+F 3 "~" H 8250 5300 50  0001 C CNN
+	1    8250 5300
+	1    0    0    -1
+$EndComp
+Text GLabel 8050 5200 0    50   Input ~ 0
+SDA
+Text GLabel 8050 5500 0    50   Input ~ 0
+SCL
+Text GLabel 8050 5300 0    50   Input ~ 0
+3v3
+Text GLabel 8050 5400 0    50   Input ~ 0
+GND
+$Comp
+L Connector:Conn_01x04_Female J3
+U 1 1 60DB9748
+P 9800 5050
+F 0 "J3" H 9828 5026 50  0000 L CNN
+F 1 "i2c Expansion" H 9828 4935 50  0000 L CNN
+F 2 "Connector_PinHeader_2.54mm:PinHeader_1x04_P2.54mm_Vertical" H 9800 5050 50  0001 C CNN
+F 3 "~" H 9800 5050 50  0001 C CNN
+	1    9800 5050
+	1    0    0    -1
+$EndComp
+Text GLabel 9600 4950 0    50   Input ~ 0
+SDA
+Text GLabel 9600 5250 0    50   Input ~ 0
+SCL
+Text GLabel 9600 5050 0    50   Input ~ 0
+3v3
+Text GLabel 9600 5150 0    50   Input ~ 0
+GND
+$Comp
+L 74xx:74HC595 U1
+U 1 1 60DD3C0F
+P 5600 1700
+F 0 "U1" H 5600 2481 50  0000 C CNN
+F 1 "74HC595" H 5600 2390 50  0000 C CNN
+F 2 "Package_SO:SOIC-16_3.9x9.9mm_P1.27mm" H 5600 1700 50  0001 C CNN
+F 3 "http://www.ti.com/lit/ds/symlink/sn74hc595.pdf" H 5600 1700 50  0001 C CNN
+	1    5600 1700
+	1    0    0    -1
+$EndComp
+$Comp
+L Jumper:SolderJumper_2_Open JP8
+U 1 1 60DD5524
+P 5050 1300
+F 0 "JP8" H 4050 1400 50  0000 C CNN
+F 1 "SolderJumper_2_Open" H 4400 1500 50  0000 C CNN
+F 2 "Jumper:SolderJumper-2_P1.3mm_Open_RoundedPad1.0x1.5mm" H 5050 1300 50  0001 C CNN
+F 3 "~" H 5050 1300 50  0001 C CNN
+	1    5050 1300
+	1    0    0    -1
+$EndComp
+$Comp
+L Jumper:SolderJumper_2_Open JP9
+U 1 1 60DDCD88
+P 5050 1500
+F 0 "JP9" H 4050 1600 50  0000 C CNN
+F 1 "SolderJumper_2_Open" H 4400 1700 50  0000 C CNN
+F 2 "Jumper:SolderJumper-2_P1.3mm_Open_RoundedPad1.0x1.5mm" H 5050 1500 50  0001 C CNN
+F 3 "~" H 5050 1500 50  0001 C CNN
+	1    5050 1500
+	1    0    0    -1
+$EndComp
+Text GLabel 5200 1600 0    50   Input ~ 0
+5V
+Text GLabel 5600 1100 1    50   Input ~ 0
+5V
+Text GLabel 5200 1900 0    50   Input ~ 0
+GND
+Text GLabel 5600 2400 3    50   Input ~ 0
+GND
+$Comp
+L Jumper:SolderJumper_2_Open JP10
+U 1 1 60DDF744
+P 5050 1800
+F 0 "JP10" H 4050 1900 50  0000 C CNN
+F 1 "SolderJumper_2_Open" H 4400 2000 50  0000 C CNN
+F 2 "Jumper:SolderJumper-2_P1.3mm_Open_RoundedPad1.0x1.5mm" H 5050 1800 50  0001 C CNN
+F 3 "~" H 5050 1800 50  0001 C CNN
+	1    5050 1800
+	1    0    0    -1
+$EndComp
+Text GLabel 3850 2350 2    50   Input ~ 0
+shift_serial
+Wire Wire Line
+	3850 2350 3550 2350
+Wire Wire Line
+	3550 2350 3550 2450
+Connection ~ 3550 2450
+Text GLabel 4900 1300 0    50   Input ~ 0
+shift_serial
+Text GLabel 4900 1500 0    50   Input ~ 0
+shift_clock
+Text GLabel 1650 2150 0    50   Input ~ 0
+shift_clock
 $EndSCHEMATC

Commit message: mass update - new blend and pcb
Parts:
- removed JP10, JP4, JP5, JP6, JP7, JP8, JP9: SolderJumper_2_Open, Jumper:SolderJumper-2_P1.3mm_Open_RoundedPad1.0x1.5mm, symbol Jumper:SolderJumper_2_Open
- removed U1: 74HC595, Package_SO:SOIC-16_3.9x9.9mm_P1.27mm, symbol 74xx:74HC595
- added J10: PG GPIO, Connector_PinHeader_2.54mm:PinHeader_1x04_P2.54mm_Vertical, symbol Connector:Conn_01x04_Female
- added J9: Audio Out, Connector_PinHeader_2.54mm:PinHeader_1x03_P2.54mm_Vertical, symbol Connector:Conn_01x03_Female
- R1, R2, R3: footprint Resistor_SMD:R_0603_1608Metric_Pad0.98x0.95mm_HandSolder -> Resistor_SMD:R_0805_2012Metric_Pad1.20x1.40mm_HandSolder
Connections:
- net 23: now also J2.16 (GPIO23)
- net 24: now also J2.18 (GPIO24)
- net 25: now also J2.22 (GPIO25)
- net 3v3: now also J10.2 (Pin_2)
- net 8: now also J2.24 (~CE0~/GPIO8)
- net GND: now also J6.3 (Pin_3), J10.1 (Pin_1), J9.3 (Pin_3)
- net button3: now also J1.36 (GPIO16); no longer J1.33 (PWM1/GPIO13)
- net ID_SD: now reaches J1.27 (ID_SD/GPIO0)
- net ID_SD: now also J2.27 (ID_SD/GPIO0)
- net ID_SC: now reaches J1.28 (ID_SC/GPIO1)
- net ID_SC: now also J2.28 (ID_SC/GPIO1)
- net audio1: now reaches J1.32 (PWM0/GPIO12)
- net audio1: now also J9.1 (Pin_1)
- net SIG: now reaches J1.38 (GPIO20/MOSI1)
- net SIG: now also J10.3 (Pin_3)
- net NS: now reaches J1.40 (GPIO21/SCLK1)
- net NS: now also J10.4 (Pin_4)
- net shift_serial: no longer names the net of J1.7 (GCLK0/GPIO4), R1.2
- new net audio2: J1.33 (PWM1/GPIO13), J9.2 (Pin_2)
Other:
- moved on the sheet: R2, R3
Changed lines of the file:
@@
 Text GLabel 3550 2650 2    50   Input ~ 0
 button2
-Text GLabel 3550 3550 2    50   Input ~ 0
+Text GLabel 1950 2150 0    50   Input ~ 0
 button3
 Text GLabel 9500 2250 2    50   Input ~ 0
@@
 Text GLabel 9500 2150 2    50   Input ~ 0
 SDA
-Text GLabel 9800 2950 2    50   Input ~ 0
+Text GLabel 9500 2950 2    50   Input ~ 0
 8
-Text GLabel 6850 3250 0    50   Input ~ 0
-25
-Text GLabel 6850 3050 0    50   Input ~ 0
-23
 Text GLabel 3850 2450 2    50   Input ~ 0
 LED1
-Text GLabel 1650 3450 0    50   Input ~ 0
+Text GLabel 1450 3450 0    50   Input ~ 0
 LED3
 $Comp
@@
 F 0 "R1" V 3493 2450 50  0000 C CNN
 F 1 "R" V 3584 2450 50  0000 C CNN
-F 2 "Resistor_SMD:R_0603_1608Metric_Pad0.98x0.95mm_HandSolder" V 3630 2450 50  0001 C CNN
+F 2 "Resistor_SMD:R_0805_2012Metric_Pad1.20x1.40mm_HandSolder" V 3630 2450 50  0001 C CNN
 F 3 "~" H 3700 2450 50  0001 C CNN
 	1    3700 2450
 	0    1    1    0
 $EndComp
-Text GLabel 1650 2250 0    50   Input ~ 0
+Text GLabel 1500 2250 0    50   Input ~ 0
 LED2
 $Comp
 L Device:R R2
 U 1 1 608FE648
-P 1800 2250
-F 0 "R2" V 1593 2250 50  0000 C CNN
-F 1 "R" V 1684 2250 50  0000 C CNN
-F 2 "Resistor_SMD:R_0603_1608Metric_Pad0.98x0.95mm_HandSolder" V 1730 2250 50  0001 C CNN
-F 3 "~" H 1800 2250 50  0001 C CNN
-	1    1800 2250
+P 1650 2250
+F 0 "R2" V 1750 2250 50  0000 C CNN
+F 1 "R" V 1650 2250 50  0000 C CNN
+F 2 "Resistor_SMD:R_0805_2012Metric_Pad1.20x1.40mm_HandSolder" V 1580 2250 50  0001 C CNN
+F 3 "~" H 1650 2250 50  0001 C CNN
+	1    1650 2250
 	0    1    1    0
 $EndComp
 Text GLabel 1950 1950 0    50   Input ~ 0
 SC_LED
-Text GLabel 6850 3150 0    50   Input ~ 0
-24
-$Comp
-L Jumper:SolderJumper_2_Open JP6
-U 1 1 60C07218
-P 7000 3050
-F 0 "JP6" H 7000 3255 50  0000 C CNN
-F 1 "SolderJumper_2_Open" H 7000 3164 50  0000 C CNN
-F 2 "Jumper:SolderJumper-2_P1.3mm_Open_RoundedPad1.0x1.5mm" H 7000 3050 50  0001 C CNN
-F 3 "~" H 7000 3050 50  0001 C CNN
-	1    7000 3050
-	1    0    0    -1
-$EndComp
-Wire Wire Line
-	7150 3050 7900 3050
-$Comp
-L Jumper:SolderJumper_2_Open JP7
-U 1 1 60C08660
-P 7000 3150
-F 0 "JP7" H 7000 3355 50  0000 C CNN
-F 1 "SolderJumper_2_Open" H 7000 3264 50  0000 C CNN
-F 2 "Jumper:SolderJumper-2_P1.3mm_Open_RoundedPad1.0x1.5mm" H 7000 3150 50  0001 C CNN
-F 3 "~" H 7000 3150 50  0001 C CNN
-	1    7000 3150
-	1    0    0    -1
-$EndComp
-Wire Wire Line
-	7900 3150 7150 3150
-$Comp
-L Jumper:SolderJumper_2_Open JP5
-U 1 1 60C09276
-P 7000 3250
-F 0 "JP5" H 7000 3455 50  0000 C CNN
-F 1 "SolderJumper_2_Open" H 7000 3364 50  0000 C CNN
-F 2 "Jumper:SolderJumper-2_P1.3mm_Open_RoundedPad1.0x1.5mm" H 7000 3250 50  0001 C CNN
-F 3 "~" H 7000 3250 50  0001 C CNN
-	1    7000 3250
-	1    0    0    -1
-$EndComp
-Wire Wire Line
-	7150 3250 7900 3250
-$Comp
-L Jumper:SolderJumper_2_Open JP4
-U 1 1 60C09F44
-P 9650 2950
-F 0 "JP4" H 9650 3155 50  0000 C CNN
-F 1 "SolderJumper_2_Open" H 9650 3064 50  0000 C CNN
-F 2 "Jumper:SolderJumper-2_P1.3mm_Open_RoundedPad1.0x1.5mm" H 9650 2950 50  0001 C CNN
-F 3 "~" H 9650 2950 50  0001 C CNN
-	1    9650 2950
-	1    0    0    -1
-$EndComp
 Text GLabel 3550 2950 2    50   Input ~ 0
 8
@@
 L Device:R R3
 U 1 1 608FB86F
-P 1800 3450
-F 0 "R3" V 1593 3450 50  0000 C CNN
-F 1 "R" V 1684 3450 50  0000 C CNN
-F 2 "Resistor_SMD:R_0603_1608Metric_Pad0.98x0.95mm_HandSolder" V 1730 3450 50  0001 C CNN
-F 3 "~" H 1800 3450 50  0001 C CNN
-	1    1800 3450
+P 1600 3450
+F 0 "R3" V 1393 3450 50  0000 C CNN
+F 1 "R" V 1484 3450 50  0000 C CNN
+F 2 "Resistor_SMD:R_0805_2012Metric_Pad1.20x1.40mm_HandSolder" V 1530 3450 50  0001 C CNN
+F 3 "~" H 1600 3450 50  0001 C CNN
+	1    1600 3450
 	0    1    1    0
 $EndComp
@@
 Text GLabel 9600 5150 0    50   Input ~ 0
 GND
-$Comp
-L 74xx:74HC595 U1
-U 1 1 60DD3C0F
-P 5600 1700
-F 0 "U1" H 5600 2481 50  0000 C CNN
-F 1 "74HC595" H 5600 2390 50  0000 C CNN
-F 2 "Package_SO:SOIC-16_3.9x9.9mm_P1.27mm" H 5600 1700 50  0001 C CNN
-F 3 "http://www.ti.com/lit/ds/symlink/sn74hc595.pdf" H 5600 1700 50  0001 C CNN
-	1    5600 1700
-	1    0    0    -1
-$EndComp
-$Comp
-L Jumper:SolderJumper_2_Open JP8
-U 1 1 60DD5524
-P 5050 1300
-F 0 "JP8" H 4050 1400 50  0000 C CNN
-F 1 "SolderJumper_2_Open" H 4400 1500 50  0000 C CNN
-F 2 "Jumper:SolderJumper-2_P1.3mm_Open_RoundedPad1.0x1.5mm" H 5050 1300 50  0001 C CNN
-F 3 "~" H 5050 1300 50  0001 C CNN
-	1    5050 1300
-	1    0    0    -1
-$EndComp
-$Comp
-L Jumper:SolderJumper_2_Open JP9
-U 1 1 60DDCD88
-P 5050 1500
-F 0 "JP9" H 4050 1600 50  0000 C CNN
-F 1 "SolderJumper_2_Open" H 4400 1700 50  0000 C CNN
-F 2 "Jumper:SolderJumper-2_P1.3mm_Open_RoundedPad1.0x1.5mm" H 5050 1500 50  0001 C CNN
-F 3 "~" H 5050 1500 50  0001 C CNN
-	1    5050 1500
-	1    0    0    -1
-$EndComp
-Text GLabel 5200 1600 0    50   Input ~ 0
-5V
-Text GLabel 5600 1100 1    50   Input ~ 0
-5V
-Text GLabel 5200 1900 0    50   Input ~ 0
-GND
-Text GLabel 5600 2400 3    50   Input ~ 0
-GND
-$Comp
-L Jumper:SolderJumper_2_Open JP10
-U 1 1 60DDF744
-P 5050 1800
-F 0 "JP10" H 4050 1900 50  0000 C CNN
-F 1 "SolderJumper_2_Open" H 4400 2000 50  0000 C CNN
-F 2 "Jumper:SolderJumper-2_P1.3mm_Open_RoundedPad1.0x1.5mm" H 5050 1800 50  0001 C CNN
-F 3 "~" H 5050 1800 50  0001 C CNN
-	1    5050 1800
-	1    0    0    -1
-$EndComp
-Text GLabel 3850 2350 2    50   Input ~ 0
-shift_serial
 Wire Wire Line
-	3850 2350 3550 2350
+	1800 2250 1950 2250
 Wire Wire Line
-	3550 2350 3550 2450
-Connection ~ 3550 2450
-Text GLabel 4900 1300 0    50   Input ~ 0
-shift_serial
-Text GLabel 4900 1500 0    50   Input ~ 0
-shift_clock
-Text GLabel 1650 2150 0    50   Input ~ 0
-shift_clock
+	1750 3450 1950 3450
+Text GLabel 3550 3450 2    50   Input ~ 0
+audio1
+Text GLabel 3550 3550 2    50   Input ~ 0
+audio2
+Text GLabel 3550 1850 2    50   Input ~ 0
+ID_SD
+Text GLabel 3550 1950 2    50   Input ~ 0
+ID_SC
+Text GLabel 9500 1850 2    50   Input ~ 0
+ID_SD
+Text GLabel 9500 1950 2    50   Input ~ 0
+ID_SC
+Text GLabel 5550 6600 0    50   Input ~ 0
+GND
+$Comp
+L Connector:Conn_01x03_Female J9
+U 1 1 61E8A339
+P 5750 6500
+F 0 "J9" H 5778 6526 50  0000 L CNN
+F 1 "Audio Out" H 5778 6435 50  0000 L CNN
+F 2 "Connector_PinHeader_2.54mm:PinHeader_1x03_P2.54mm_Vertical" H 5750 6500 50  0001 C CNN
+F 3 "~" H 5750 6500 50  0001 C CNN
+	1    5750 6500
+	1    0    0    -1
+$EndComp
+Text GLabel 5550 6400 0    50   Input ~ 0
+audio1
+Text GLabel 5550 6500 0    50   Input ~ 0
+audio2
+Text GLabel 3250 6500 0    50   Input ~ 0
+GND
+Text GLabel 7900 3050 0    50   Input ~ 0
+23
+Text GLabel 7900 3150 0    50   Input ~ 0
+24
+Text GLabel 7900 3250 0    50   Input ~ 0
+25
+Text GLabel 1950 2650 0    50   Input ~ 0
+SIG
+Text GLabel 1950 2750 0    50   Input ~ 0
+NS
+$Comp
+L Connector:Conn_01x04_Female J10
+U 1 1 61F15261
+P 7050 5300
+F 0 "J10" H 7078 5276 50  0000 L CNN
+F 1 "PG GPIO" H 7078 5185 50  0000 L CNN
+F 2 "Connector_PinHeader_2.54mm:PinHeader_1x04_P2.54mm_Vertical" H 7050 5300 50  0001 C CNN
+F 3 "~" H 7050 5300 50  0001 C CNN
+	1    7050 5300
+	1    0    0    -1
+$EndComp
+Text GLabel 6850 5300 0    50   Input ~ 0
+3v3
+Text GLabel 6850 5200 0    50   Input ~ 0
+GND
+Text GLabel 6850 5400 0    50   Input ~ 0
+SIG
+Text GLabel 6850 5500 0    50   Input ~ 0
+NS
 $EndSCHEMATC
